Commit message: Implements urdf model of robot but can't use cad files bc 2017a

File: src/my_robot.urdf (robot description, URDF)
Before this commit: robot test_robot, 4 links, 3 joints
Links:
- link link0: geometry visual mesh filename=/ifs/home/jwternent/RBE3001_Matlab01/src/CAD/Link0.stl
Joints:
- joint joint1: type fixed -> continuous
